File: System Controller/SystemController.sch (KiCad schematic (older format))
At the start: 60 parts, among them P1 Battery Input, P2 SWD, P3 Raspberry Pi A+ Connectors, P4 Harwin-10P, P5 Harwin-10P, P6 Harwin-10P, Q1 2N7002, Q2 Si2343CDS, SW1 SW_PUSH, U1 LM317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

Commit message: Refactoring local repository.
Other:
- note added: "Motor Connections\n"
- note added: "RPi A+ Connections\n"
- moved on the sheet: P3, P4, P5, P6
