File: Electronics/System Controller/SystemController.kicad_pcb (KiCad board)
At the start: 2 copper layers, 65 x 56 mm, 61 parts, among them P1 Battery Input, P2 SWD, P3 Raspberry Pi A+ Connectors, P4 Harwin-10P, P5 Harwin-10P, P6 Harwin-10P, Q1 2N7002, Q2 Si2343CDS, SW1 SW_PUSH, U1 LM317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

Commit message: PCB Tidy-up
Slight changes to SystemController PCB
Parts:
- moved G*** 6.74 mm to (72.5, 107.9)
Other:
- board text added: "Design: Nathan Perkins"
- board text added: "Yatagarasu v1.0"
- board text removed: "Yatagarasu v1.0 Nathan Perkins"
Changed lines of the file:
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@@
-(kicad_pcb (version 4) (host pcbnew 0.201603151217+6622~43~ubuntu15.10.1-product)
+(kicad_pcb (version 4) (host pcbnew 0.201603171416+6624~43~ubuntu15.10.1-product)
   (general
     (links 162)
     (no_connects 1)
-    (area 57.384999 85.324999 122.535015 141.475001)
+    (area 57.384999 70.05 138.075 145.045001)
     (thickness 1.6)
-    (drawings 11)
+    (drawings 12)
     (tracks 891)
     (zones 0)
@@
   )
   (layers
-    (0 F.Cu signal)
+    (0 F.Cu signal hide)
     (31 B.Cu signal)
     (32 B.Adhes user)
@@
   )
   (module NPFootprints:Yatagarsu_Logo (layer B.Cu)
-    (at 70.94 114.44 180)
+    (at 72.475 107.875 180)
     (fp_text reference G*** (at 0.08 0.81 180) (layer B.SilkS) hide
       (effects (font (thickness 0.3)) (justify mirror))
@@
       (xy -1.693333 2.421467) (xy -1.691785 2.424952) (xy -1.690511 2.424289)) (layer B.SilkS) (width 0.01))
   )
+  (gr_text "Design: Nathan Perkins" (at 68.409523 102.325) (layer B.SilkS)
+    (effects (font (size 1 1) (thickness 0.1875)) (justify mirror))
+  )
   (dimension 65 (width 0.3) (layer Margin)
     (gr_text "65.000 mm" (at 89.95 71.4) (layer Margin)
@@
   (gr_line (start 122.46 137.9) (end 122.46 88.9) (angle 90) (layer Edge.Cuts) (width 0.15))
   (gr_line (start 60.96 141.4) (end 118.96 141.4) (angle 90) (layer Edge.Cuts) (width 0.15))
-  (gr_text "Yatagarasu v1.0\nNathan Perkins" (at 73 102.4) (layer B.SilkS)
+  (gr_text "Yatagarasu v1.0" (at 68.1 100.1) (layer B.SilkS)
     (effects (font (size 1.5 1.5) (thickness 0.3)) (justify mirror))
   )
